Commit message: lab2 finalne

File: src/lab2_robot/urdf/moving_robot.urdf (robot description, URDF)
Before this commit: robot example_robot, 4 links, 3 joints
Joints:
- joint base_to_link1: axis (none) -> 0 0 1; limit (none) -> lower=-${data['row1']['l_len']} upper=0 effort=1000.0 velocity=0.5; type fixed -> prismatic
- joint link1_to_link2: axis (none) -> 0 0 1; limit (none) -> lower=-${data['row2']['l_len']} upper=0 effort=1000.0 velocity=0.5; type fixed -> prismatic
- joint link2_to_link3: axis (none) -> 0 0 1; limit (none) -> lower=-${data['row3']['l_len']} upper=0 effort=1000.0 velocity=0.5; type fixed -> prismatic

Commit message: dodana sfera

File: src/lab2_robot/urdf/moving_robot.urdf (robot description, URDF)
Before this commit: robot example_robot, 4 links, 3 joints
Links:
- added link link_4; visual sphere radius=0.1
Joints:
- added joint link3_to_link4: type fixed, parent link_3, child link_4, origin xyz=0 0 0 rpy=0 0 0

File: src/lab2_robot/urdf/static_robot.urdf (robot description, URDF)
Before this commit: robot example_robot, 4 links, 3 joints
Links:
- added link link_4; visual sphere radius=0.1
Joints:
- added joint link3_to_link4: type fixed, parent link_3, child link_4, origin xyz=0 0 0 rpy=0 0 0
